File: Hardware/battery_box/battery_box.sch (EAGLE design)
At the start: 45 parts, among them IC1 AD826R, J1 CON_HEADER_PRG_PIC_ICSPA, Q1 IRFR5505PBFTO252, Q2 BSS123, X1 CON_MOLEX_39_29_1028, X2 KUSBVX

Commit message: First PCB Layout
Parts:
- removed U$1: EQUINOX_LOGO_SMALL, equinox:EQUINOX_LOGO_SMALL
Changed lines of the file:
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@@
 <?xml version="1.0" encoding="utf-8"?>
 <!DOCTYPE eagle SYSTEM "eagle.dtd">
-<eagle version="6.3">
+<eagle version="6.4">
 <drawing>
 <settings>
@@
 <part name="R18" library="rcl" deviceset="R-EU_" device="R0805" value="1M"/>
 <part name="R19" library="rcl" deviceset="R-EU_" device="R0805" value="10k"/>
-<part name="U$1" library="equinox" deviceset="EQUINOX_LOGO_SMALL" device=""/>
 <part name="DATA_OUT" library="con-lstb" deviceset="MA04-1" device=""/>
 </parts>
@@
 <instance part="R18" gate="G$1" x="160.02" y="170.18" rot="R270"/>
 <instance part="R19" gate="G$1" x="78.74" y="114.3" rot="R90"/>
-<instance part="U$1" gate="G$1" x="314.96" y="12.7"/>
 <instance part="DATA_OUT" gate="1" x="68.58" y="22.86"/>
 </instances>

Commit message: Updated the DC Jack and Battery Connector
Fixed problems with footprints
Parts:
- added U$1: EQUINOX_LOGO_SMALL, equinox:EQUINOX_LOGO_SMALL
Other:
- note removed: "2069436"
- note removed: "Added e.quinox logo"
- note removed: "Change for low power voltage regulator"
- note removed: "Change to 3.3V"
- note removed: "Need to change to cheaper op amp"
Changed lines of the file:
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@@
 <?xml version="1.0" encoding="utf-8"?>
 <!DOCTYPE eagle SYSTEM "eagle.dtd">
-<eagle version="6.4">
+<eagle version="6.3">
 <drawing>
 <settings>
@@
 <layers>
 <layer number="1" name="Top" color="4" fill="1" visible="no" active="no"/>
+<layer number="2" name="Route2" color="1" fill="3" visible="no" active="no"/>
+<layer number="3" name="Route3" color="4" fill="3" visible="no" active="no"/>
+<layer number="4" name="Route4" color="1" fill="4" visible="no" active="no"/>
+<layer number="5" name="Route5" color="4" fill="4" visible="no" active="no"/>
+<layer number="6" name="Route6" color="1" fill="8" visible="no" active="no"/>
+<layer number="7" name="Route7" color="4" fill="8" visible="no" active="no"/>
+<layer number="8" name="Route8" color="1" fill="2" visible="no" active="no"/>
+<layer number="9" name="Route9" color="4" fill="2" visible="no" active="no"/>
+<layer number="10" name="Route10" color="1" fill="7" visible="no" active="no"/>
+<layer number="11" name="Route11" color="4" fill="7" visible="no" active="no"/>
+<layer number="12" name="Route12" color="1" fill="5" visible="no" active="no"/>
+<layer number="13" name="Route13" color="4" fill="5" visible="no" active="no"/>
+<layer number="14" name="Route14" color="1" fill="6" visible="no" active="no"/>
+<layer number="15" name="Route15" color="4" fill="6" visible="no" active="no"/>
 <layer number="16" name="Bottom" color="1" fill="1" visible="no" active="no"/>
 <layer number="17" name="Pads" color="2" fill="1" visible="no" active="no"/>
@@
 <part name="R19" library="rcl" deviceset="R-EU_" device="R0805" value="10k"/>
 <part name="DATA_OUT" library="con-lstb" deviceset="MA04-1" device=""/>
+<part name="U$1" library="equinox" deviceset="EQUINOX_LOGO_SMALL" device=""/>
 </parts>
 <sheets>
 <sheet>
 <plain>
-<text x="45.72" y="88.9" size="1.778" layer="98" rot="R90">Change for low power voltage regulator</text>
 <text x="20.32" y="167.64" size="1.778" layer="98" rot="R270">Molex connector to crimped battery</text>
 <text x="190.5" y="7.62" size="1.778" layer="98">PCB Mounts</text>
-<text x="294.64" y="27.94" size="1.778" layer="98">Added e.quinox logo</text>
-<text x="45.72" y="66.04" size="1.778" layer="98" rot="R90">Change to 3.3V</text>
-<text x="43.18" y="66.04" size="1.778" layer="98" rot="R90">2069436</text>
-<text x="190.5" y="116.84" size="3.81" layer="98">Need to change to cheaper op amp</text>
 </plain>
 <instances>
@@
 <instance part="R19" gate="G$1" x="78.74" y="114.3" rot="R90"/>
 <instance part="DATA_OUT" gate="1" x="68.58" y="22.86"/>
+<instance part="U$1" gate="G$1" x="314.96" y="12.7"/>
 </instances>
 <busses>
