File: Hardware/battery_box/Battery_Box_2013_v3/battery_box3.brd (EAGLE design)
At the start: 60 x 80 mm, 54 parts, among them IC1 AD826R, IC2 LM2574, IC3 PIC16F1824, IC4 LD117AS18TR, J1 CON_HEADER_PRG_PIC_ICSPA, Q1 IRFR5505PBFTO252, Q2 BSS123, X1 CON_MOLEX_39_29_1028

Commit message: Added Battery Box V3
Parts:
- removed C8: 10u, 6.3V, rcl:C0805
- removed D3: (no value), diode:SMC
- removed U$1: EQUINOX_LOGO_SMALL, equinox:EQUINOX_LOGO_SMALL
- added C7: 10u, 6.3V, rcl:C0805
- TP2: value TPTP14R -> TPTP20R; device testpad:TP14R -> testpad:TP20R
- moved D2 49.6 mm to (5.00, 44.0), turned to 270 degrees
- moved TP2 8.60 mm to (55.0, 62.0)
- moved IC4 2.24 mm to (45.0, 71.0)
- moved D1 1.00 mm to (14.0, 6.00)
- renumbered X1 to X1CON
Connections:
- net 12V_OUT: no longer D2.A
- net GND: now also C7.2, D2.A; no longer C8.2, D3.A
- net VDD: now also C7.1; no longer C8.1
- net V_BATT: no longer D3.C
Routing:
- net 12V_OUT: track 103.6 -> 89.9 mm
- net PGD: track 25.0 -> 31.1 mm
- net PGC: track 27.2 -> 30.3 mm
- net V_BATT: track 132.1 -> 134.6 mm
- net GND: track 108.8 -> 107.8 mm
- net VDD: track 64.8 -> 65.7 mm
Other:
- board text added: "X1Con"
